File: PCB/main-board/main-board.kicad_pcb (KiCad board)
At the start: 2 copper layers, 185 x 82 mm, 114 parts, among them J1 USB_C_Receptacle_USB2.0_16P, SW1 BOOT, SW2 REC/STOP, SW3 RESET, U1 LM393, U10 74AHCT125, U11 ITR8307-S17-TR8, U12 ITR8307-S17-TR8, U13 USBLC6-2SC6, U14 RP2040, U15 AMS1117-3.3, U16 W25Q16JVSS, U2 LM358, U3 LM358, U4 LM393, U5 GS3011C, U6 GS3011C, U7 GS3011C, U8 MAX7219, U9 ITR8307-S17-TR8, Y1 12MHz 20pF 50Ohm_ESR

Commit message: v1.1 as ordered
Parts:
- removed the G*** at (169.5, 130.5)
- removed the G*** at (189.4, 125.7)
- removed kibuzzard-6930AFAB: G***, kibuzzard-6930AFAB
- removed kibuzzard-69310240: G***, kibuzzard-69310240
- removed kibuzzard-6964435B: G***, kibuzzard-6964435B
- removed kibuzzard-6978203B: G***, kibuzzard-6978203B
- removed kibuzzard-6978204E: G***, kibuzzard-6978204E
- removed kibuzzard-697836DA: G***, kibuzzard-697836DA
- removed kibuzzard-6978422B: G***, kibuzzard-6978422B
- removed kibuzzard-69784254: G***, kibuzzard-69784254
- removed kibuzzard-697848C9: G***, kibuzzard-697848C9
- added G***: LOGO, LOGO, F.Cu at (132.2, 116.5)
- added G***: LOGO, LOGO, F.Cu at (169.6, 130.5)
- added G***: LOGO, LOGO, F.Cu at (189.1, 114.1)
- added kibuzzard-6A5D9600: G***, kibuzzard-6A5D9600, F.Cu at (218.8, 134.0)
- added kibuzzard-6A5D9E3D: G***, kibuzzard-6A5D9E3D, B.Cu at (197.2, 130.7)
- added kibuzzard-6A5DA214: G***, kibuzzard-6A5DA214, F.Cu at (169.5, 123.8)
- added kibuzzard-6A5DFDED: G***, kibuzzard-6A5DFDED, F.Cu at (115.2, 135.2)
- added kibuzzard-6A5DFE62: G***, kibuzzard-6A5DFE62, F.Cu at (192.7, 140.5)
- added kibuzzard-6A601CB9: G***, kibuzzard-6A601CB9, F.Cu at (60.8, 121.2)
- added kibuzzard-6A601CBF: G***, kibuzzard-6A601CBF, F.Cu at (80.8, 121.0)
- added kibuzzard-6A601CD4: G***, kibuzzard-6A601CD4, F.Cu at (46.2, 129.2)
- moved U10 17.9 mm to (167.5, 122.5), turned to 0 degrees
- moved U5 12.3 mm to (123.5, 135.1)
- moved U6 12.3 mm to (131.7, 135.1)
- moved U7 12.3 mm to (139.9, 135.1)
- moved kibuzzard-6930AF86 8.50 mm to (147.8, 137.5)
- moved C22 3.30 mm to (158.8, 124.5)
- moved R2 3.30 mm to (158.8, 122.7)
- moved R3 3.30 mm to (158.8, 121.1)
- moved U8 3.30 mm to (151.1, 122.4)
- moved H10 1.00 mm to (44.2, 140.0)
- moved H11 1.00 mm to (44.2, 109.0)
- moved H12 1.00 mm to (219.2, 109.0)
- moved H9 1.00 mm to (219.2, 140.0)
- moved REF** 0.70 mm to (170.4, 140.5)
Connections:
- U10 pad 11: unconnected-(U10-Pad11) -> Net-(U8-DIN)
- U10 pad 12: GND -> /7SEG_DATA
- U10 pad 2: /7SEG_~{CS} -> /7SEG_CLK
- U10 pad 3: Net-(U8-LOAD) -> Net-(U8-CLK)
- U10 pad 5: /7SEG_CLK -> /7SEG_~{CS}
- U10 pad 6: Net-(U8-CLK) -> Net-(U8-LOAD)
- U10 pad 8: Net-(U8-DIN) -> unconnected-(U10-Pad8)
- U10 pad 9: /7SEG_DATA -> GND
Routing:
- net /7SEG_DATA: track 55.9 -> 97.2 mm
- net /7SEG_~{CS}: track 63.1 -> 96.9 mm
- net /7SEG_CLK: track 57.5 -> 89.6 mm
- net Net-(U8-DIN): track 4.39 -> 30.0 mm, vias 0 -> 2
- net Net-(U8-LOAD): track 43.5 -> 22.6 mm
- net Net-(U8-CLK): track 31.7 -> 14.8 mm
- net /DP: track 45.8 -> 59.9 mm
- net /E: track 52.7 -> 63.3 mm, vias 5 -> 3
- net +5V: track 187.7 -> 195.2 mm
- net /G: track 59.2 -> 52.2 mm, vias 3 -> 4
- net /F: track 45.4 -> 50.6 mm
- net /C: track 46.5 -> 51.6 mm
- net /D: track 55.4 -> 59.8 mm
- net /A: track 58.2 -> 55.4 mm
- net GND: track 144.8 -> 143.0 mm, vias 36 -> 38
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Other:
- board size 185 x 82 mm -> 185 x 83 mm
- board text added: "Design by michaelruppe.com 2026"
- board text removed: "Design by Michael Ruppe 2026"
- board text removed: "Designed at Monash University in partnership with MathWorks®"

Commit message: update design with lessons learned from pilot production
Parts:
- removed R1, R4: 1k, Resistor_SMD:R_0603_1608Metric
- removed R12, R5: 10k, Resistor_SMD:R_0603_1608Metric
- removed kibuzzard-6A5D9600: G***, kibuzzard-6A5D9600
- added C23: 100nF, Capacitor_SMD:C_0603_1608Metric, B.Cu at (172.5, 125.8)
- added R26: 10k, Resistor_SMD:R_0603_1608Metric, B.Cu at (184.7, 75.8)
- added R33: 10k, Resistor_SMD:R_0603_1608Metric, B.Cu at (184.7, 73.8)
- added R34: 10k, Resistor_SMD:R_0603_1608Metric, B.Cu at (184.7, 77.8)
- added kibuzzard-6A754149: G***, kibuzzard-6A754149, F.Cu at (218.8, 134.0)
- added kibuzzard-6A815F94: G***, kibuzzard-6A815F94, B.Cu at (66.5, 142.8)
- R7: value 10k -> 1k
- moved R7 1.78 mm to (184.7, 79.6), turned to 180 degrees
- moved G*** 0.25 mm to (197.3, 122.8)
Connections:
- C1 pad 1: +3V3 -> +5V
- C2 pad 1: +3V3 -> +5V
- C3 pad 1: +3V3 -> +5V
- C4 pad 1: +3V3 -> +5V
- R7 pad 1: Net-(R5-Pad2) -> GND
- U1 pad 8: +3V3 -> +5V
- U2 pad 8: +3V3 -> +5V
- U3 pad 8: +3V3 -> +5V
- U4 pad 8: +3V3 -> +5V
Routing:
- net +5V: track 195.2 -> 254.3 mm, vias 2 -> 8
- net +3V3: track 64.6 -> 51.1 mm, vias 3 -> 1
- net GND: track 143.0 -> 138.2 mm
- net /V_REF: track 35.9 -> 39.0 mm
- net Net-(R4-Pad1): track 2.43 -> 0.00 mm
- net Net-(R5-Pad2): track 2.43 -> 0.00 mm
- net Net-(R1-Pad1): track 2.43 -> 0.00 mm
- net Net-(U8-LOAD): track 22.6 -> 21.3 mm
- net /~{BOOT}: track 40.0 -> 40.9 mm
- net /PHOTO_A: track 107.1 -> 107.9 mm
- net /7SEG_~{CS}: track 96.9 -> 97.4 mm
- net Net-(U8-CLK): track 14.8 -> 14.3 mm
Other:
- board text removed: "Design by michaelruppe.com 2026"

Commit message: v2.0 PCB as ordered
Parts:
- removed C9: 100nF, Capacitor_SMD:C_0603_1608Metric
- removed R7: 1k, Resistor_SMD:R_0603_1608Metric
- removed kibuzzard-6A754149: G***, kibuzzard-6A754149
- added C24: 1uF, Capacitor_SMD:C_0603_1608Metric, B.Cu at (175.7, 95.4)
- added C25: 1uF, Capacitor_SMD:C_0603_1608Metric, B.Cu at (186.4, 84.0)
- added C26: 1uF, Capacitor_SMD:C_0603_1608Metric, B.Cu at (176.9, 80.6)
- added C27: 1uF, Capacitor_SMD:C_0603_1608Metric, B.Cu at (164.8, 91.6)
- added C28: 10uF, Capacitor_SMD:C_0603_1608Metric, B.Cu at (174.2, 125.8)
- added R12: 10k, Resistor_SMD:R_0603_1608Metric, B.Cu at (175.7, 93.8)
- added R35: 220, Resistor_SMD:R_0603_1608Metric, B.Cu at (103.8, 128.0)
- added R36: 220, Resistor_SMD:R_0603_1608Metric, B.Cu at (103.8, 129.6)
- added TP10: TestPoint, TestPoint:TestPoint_Pad_D1.5mm, B.Cu at (170.0, 98.8)
- added TP7: TestPoint, TestPoint:TestPoint_Pad_D1.5mm, B.Cu at (174.0, 81.8)
- added TP8: TestPoint, TestPoint:TestPoint_Pad_D1.5mm, B.Cu at (185.7, 82.0)
- added TP9: TestPoint, TestPoint:TestPoint_Pad_D1.5mm, B.Cu at (174.0, 98.8)
- added kibuzzard-6A9CABE9: G***, kibuzzard-6A9CABE9, F.Cu at (218.8, 134.0)
- added kibuzzard-6A9CB9E8: G***, kibuzzard-6A9CB9E8, B.Cu at (184.2, 90.5)
- added kibuzzard-6A9CBA16: G***, kibuzzard-6A9CBA16, B.Cu at (168.0, 81.8)
- added kibuzzard-6A9CBA29: G***, kibuzzard-6A9CBA29, B.Cu at (168.5, 77.8)
- added kibuzzard-6A9CBA31: G***, kibuzzard-6A9CBA31, B.Cu at (168.0, 71.8)
- added kibuzzard-6A9CBA3E: G***, kibuzzard-6A9CBA3E, B.Cu at (168.4, 90.8)
- added kibuzzard-6A9CBA47: G***, kibuzzard-6A9CBA47, B.Cu at (168.0, 94.8)
- added kibuzzard-6A9CBA92: G***, kibuzzard-6A9CBA92, B.Cu at (182.8, 82.0)
- added kibuzzard-6A9CBA99: G***, kibuzzard-6A9CBA99, B.Cu at (177.0, 98.8)
- added kibuzzard-6A9CBA9F: G***, kibuzzard-6A9CBA9F, B.Cu at (173.2, 83.3)
- added kibuzzard-6A9CBB45: G***, kibuzzard-6A9CBB45, B.Cu at (167.4, 98.8)
- C21: value 100nF -> 1uF
- R13, R18, R6: value 150k -> 330k
- R34: value 10k -> 220
- moved R34 94.3 mm to (103.8, 126.3)
- moved R33 11.5 mm to (176.8, 82.2)
- moved C21 11.3 mm to (180.8, 91.9)
- moved R26 10.2 mm to (186.4, 85.8)
- moved C17 4.90 mm to (114.2, 111.6), turned to 90 degrees
- moved C11 2.70 mm to (109.2, 118.6), turned to -90 degrees
- moved C15 1.81 mm to (97.0, 121.8)
- moved C18 1.40 mm to (111.3, 115.2)
- moved R27 1.40 mm to (108.6, 114.2)
- moved Y1 1.40 mm to (111.3, 112.2)
- moved C14 1.04 mm to (107.2, 118.6), turned to -90 degrees
- moved C13 0.71 mm to (98.2, 110.0)
- moved C2 0.07 mm to (164.8, 89.8)
Connections:
- net Net-(U2A--) renamed /BUFF_A
- net Net-(U2B--) renamed /BUFF_B
- C21 pad 1: /V_REF -> +5V
- R22 pad 1: Net-(U3A--) -> /BUFF_C
- R26 pad 1: +3V3 -> /PWM_B
- R26 pad 2: /V_REF -> /V_{refB}
- R33 pad 1: +3V3 -> /PWM_C
- R33 pad 2: /V_REF -> /V_{refC}
- R34 pad 1: +3V3 -> /BUFF_C
- R34 pad 2: /V_REF -> Net-(U14-GPIO26_ADC0)
- TP5 pad 1: Net-(U3A--) -> /BUFF_C
- U1 pad 2: /V_REF -> /V_{refA}
- U1 pad 6: /V_REF -> /V_{refB}
- U14 pad 15: unconnected-(U14-GPIO12-Pad15) -> /PWM_A
- U14 pad 16: unconnected-(U14-GPIO13-Pad16) -> /PWM_B
- U14 pad 17: unconnected-(U14-GPIO14-Pad17) -> /PWM_C
- U14 pad 2: unconnected-(U14-GPIO0-Pad2) -> /PHOTO_C
- U14 pad 3: unconnected-(U14-GPIO1-Pad3) -> /PHOTO_A
- U14 pad 37: /PHOTO_C -> unconnected-(U14-GPIO25-Pad37)
- U14 pad 38: /PHOTO_A -> Net-(U14-GPIO26_ADC0)
- U14 pad 39: /PHOTO_B -> Net-(U14-GPIO27_ADC1)
- U14 pad 4: unconnected-(U14-GPIO2-Pad4) -> /PHOTO_B
- U14 pad 40: unconnected-(U14-GPIO28_ADC2-Pad40) -> Net-(U14-GPIO28_ADC2)
- U3 pad 1: Net-(U3A--) -> /BUFF_C
- U3 pad 2: Net-(U3A--) -> /BUFF_C
- U4 pad 2: /V_REF -> /V_{refC}
Routing:
- net /PWM_C: track 0.00 -> 120.9 mm, vias 0 -> 2
- net /BUFF_C: track 0.00 -> 112.0 mm
- net /PWM_B: track 0.00 -> 100.8 mm, vias 0 -> 2
- net /BUFF_B: track 7.82 -> 101.7 mm, vias 0 -> 2
- net /PWM_A: track 0.00 -> 90.4 mm, vias 0 -> 2
- net +5V: track 254.3 -> 344.1 mm
- net /BUFF_A: track 19.4 -> 105.8 mm
- net /V_REF: track 39.0 -> 0.00 mm
- net /V_{refA}: track 0.00 -> 15.3 mm, vias 0 -> 2
- net Net-(U3A--): track 14.0 -> 0.00 mm
- net Net-(U14-GPIO28_ADC2): track 0.00 -> 12.5 mm
- net /PHOTO_C: track 116.2 -> 104.0 mm
- net /PHOTO_A: track 107.9 -> 96.1 mm, vias 0 -> 2
- net Net-(U14-GPIO27_ADC1): track 0.00 -> 10.9 mm
- net /PHOTO_B: track 116.7 -> 106.0 mm, vias 0 -> 2
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