File: PCB/main-board/main-board.kicad_sch (KiCad schematic)
At the start: 94 parts, among them J1 USB_C_Receptacle_USB2.0_16P, SW1 BOOT, SW2 REC/STOP, SW3 RESET, U1 LM393, U10 74AHCT125, U11 ITR8307-S17-TR8, U12 ITR8307-S17-TR8, U13 USBLC6-2SC6, U14 RP2040, U15 AMS1117-3.3, U16 W25Q16JVSS, U2 LM358, U3 LM358, U4 LM393, U5 GS3011C, U6 GS3011C, U7 GS3011C, U8 MAX7219, U9 ITR8307-S17-TR8, Y1 12MHz 20pF 50Ohm_ESR

Commit message: v1.1 as ordered
Parts:
- TP1, TP2, TP3, TP4, TP5, TP6: now left out of the parts list
Connections:
- net 7SEG_CLK: now also U10.2; no longer U10.5
- net 7SEG_DATA: now also U10.12; no longer U10.9
- net 7SEG_~{CS}: now also U10.5; no longer U10.2
- net GND: now also U10.9; no longer U10.12
- net at U10.11: now also U8.1 (DIN)
- net at U10.8: no longer U8.1 (DIN)
- net at U10.3: now also U8.13 (CLK); no longer U8.12 (LOAD)
- net at U10.6: now also U8.12 (LOAD); no longer U8.13 (CLK)

Commit message: update design with lessons learned from pilot production
Parts:
- removed R1, R4: 1k, Resistor_SMD:R_0603_1608Metric, symbol Device:R
- removed R12, R5: 10k, Resistor_SMD:R_0603_1608Metric, symbol Device:R
- added C23: 100nF, Capacitor_SMD:C_0603_1608Metric, symbol Device:C
- added R26, R33, R34: 10k, Resistor_SMD:R_0603_1608Metric, symbol Device:R
- R7: value 10k -> 1k; LCSC Part # C25804 -> C21190
Connections:
- net +3V3: now also R26.1, R33.1, R34.1; no longer C1.1, C2.1, C3.1, C4.1, U1.8 (V+), U2.8 (V+), U3.8 (V+), U4.8 (V+)
- net +5V: now also C1.1, C2.1, C3.1, C4.1, U1.8 (V+), U2.8 (V+), U3.8 (V+), U4.8 (V+), C23.1
- net GND: now also R7.1, C23.2
- net V_REF: now also R26.2, R33.2, R34.2
Other:
- note added: "Components reused to optimise BOM."
- note added: "Spare"
- note added: "V_{ref} = 0.76V"
- note removed: "Components reused to optimise BOM. Use 1V reference if desired"
- note removed: "Hi Thresh: 1.1V Lo Thresh: 0.9V"
- note removed: "V_{ref} = 1.03V"
- moved on the sheet: C1, C2, C21, C3, C4, R10, R11, R13, R14, R15, R16, R17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

Commit message: v2.0 PCB as ordered
Parts:
- removed C9: 100nF, Capacitor_SMD:C_0603_1608Metric, symbol Device:C
- removed R7: 1k, Resistor_SMD:R_0603_1608Metric, symbol Device:R
- added C24, C25, C26, C27: 1uF, Capacitor_SMD:C_0603_1608Metric, symbol Device:C
- added C28: 10uF, Capacitor_SMD:C_0603_1608Metric, symbol Device:C
- added R12: 10k, Resistor_SMD:R_0603_1608Metric, symbol Device:R
- added R35, R36: 220, Resistor_SMD:R_0603_1608Metric, symbol Device:R
- added TP10, TP7, TP8, TP9: TestPoint, TestPoint:TestPoint_Pad_D1.5mm, symbol Connector:TestPoint
- C21: value 100nF -> 1uF; LCSC Part # C14663 -> C15849
- R13, R18, R6: value 150k -> 330k; LCSC Part # C22807 -> C23137
- R34: value 10k -> 220; LCSC Part # C25804 -> C22962
Connections:
- net +3V3: no longer R26.1, R33.1, R34.1
- net +5V: now also C21.1, C27.1, C28.1
- net GND: now also C24.2, C25.2, C26.2, C27.2, C28.2, TP10.1
- net PHOTO_A: now also U14.3 (GPIO1); no longer U14.38 (GPIO26_ADC0)
- net PHOTO_B: now also U14.4 (GPIO2); no longer U14.39 (GPIO27_ADC1)
- net PHOTO_C: now also U14.2 (GPIO0); no longer U14.37 (GPIO25)
- net BUFF_C: now reaches R22.1, TP5.1, U3.1, U3.2 (-)
- net BUFF_C: now also R34.1
- net BUFF_B: now reaches R17.1, TP3.1, U2.6 (-), U2.7
- net BUFF_B: now also R36.2
- net BUFF_A: now reaches R11.1, TP1.1, U2.1, U2.2 (-)
- net BUFF_A: now also R35.2
- net PWM_A: now reaches U14.15 (GPIO12)
- net PWM_A: now also R12.1
- net PWM_B: now reaches U14.16 (GPIO13)
- net PWM_B: now also R26.1
- net PWM_C: now reaches U14.17 (GPIO14)
- net PWM_C: now also R33.1
- net at U14.40 (GPIO28_ADC2): now also R36.1
- removed net V_REF: C21.1, R26.2, R33.2, R34.2, U1.2 (-), U1.6 (-), U4.2 (-)
- new net: R34.2, U14.38 (GPIO26_ADC0)
- new net: R35.1, U14.39 (GPIO27_ADC1)
- new net V_{refA}: C24.1, R12.2, TP9.1, U1.2 (-)
- new net V_{refB}: C25.1, R26.2, TP8.1, U1.6 (-)
- new net V_{refC}: C26.1, R33.2, TP7.1, U4.2 (-)
- no-connect marks 35 -> 29
Other:
- note added: "Per-channel voltage reference accounts for variation between IR reflectance sensors"
- note added: "Place RC filter close to comparator"
- note removed: "Components reused to optimise BOM."
- note removed: "V_{ref} = 0.76V"
- moved on the sheet: C1, C10, C11, C12, C13, C14, C15, C16, C17, C18, C2, C22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
